File: hardware/TV_Lift_Kicad files/_autosave-controller_Tv_Lift.kicad_pcb (KiCad board)
At the start: 4 copper layers, 70 x 157.5 mm, 96 parts, among them J1 socket LAN8720a, J10 CONN_IR_OUT, J11 DRY CONTACT UP DOWN, J12 DRY CONTACT, J2 POWER 24V, J3 CAN_bus, J4 ENCODER, J5 ENCODER_POWER, J6 CONN_RS232, J7 M1 LIMIT UP DOWN, J8 Signal PWR, J9 MOTOR_OUT, Q1 2N3904, SW1 UP, SW2 DOWN, SW3 STOP, U1 MAX3232, U10 VNH5019A-E, U2 TSOP32S40F, U3 SN65HVD230, U4 ESP32-WROOM-32, U5 LM2596S-5, U6 AMS1117-3.3, U7 PC817, U8 PC817, U9 NCS1S1205SC

Commit message: fix schema ( fuse + annotation)
Parts:
- F1: value Fuse_Small -> Fuse_Mini_10A
- LED1: renamed from LED_GREEN_F3_POWER1; value LED -> LED_GREEN_F3
- LED2: renamed from LED_RED_F3_ERROR1; value LED_ERROR -> LED_RED_F3
- moved J2 1.50 mm to (73.9, 53.8)
- moved R22 1.41 mm to (122.5, 161.5), turned to -90 degrees
- moved R27 1.33 mm to (116.5, 161.6), turned to -90 degrees
- moved C6 1.12 mm to (115.0, 167.0)
- moved C10 0.59 mm to (121.8, 166.0)
- moved Q1 0.40 mm to (121.5, 156.3)
- moved J10 0.06 mm to (127.1, 158.8)
- renumbered D3 to LED3
Routing:
- net Net-(J2-Pin_1): track 34.1 -> 38.7 mm
- net Net-(J10-Pin_2): track 6.58 -> 9.22 mm
- net Net-(J10-Pin_1): track 5.56 -> 7.05 mm
- net +5V: track 187.5 -> 188.4 mm, vias 6 -> 7
- net Net-(U4-EN): track 13.0 -> 13.8 mm
- net +3.3V: track 71.9 -> 72.4 mm
- net GNDPWR: vias 43 -> 42
- net +24V: vias 10 -> 11
Other:
- board text added: "+"
- board text added: "+24"
- board text added: "+3.3V"
- board text added: "-"
- board text added: "- (GND)"
- board text added: "CANH"
- board text added: "CANL"
- board text added: "IR EMMITER: + : STRIPE (ANOD) - : BLACK (KATOD)"
