File: hardware/TV_Lift_Kicad files/_autosave-controller_Tv_Lift.kicad_sch (KiCad schematic)
At the start: 96 parts, among them J1 socket LAN8720a, J10 CONN_IR_OUT, J11 DRY CONTACT UP DOWN, J12 DRY CONTACT, J2 POWER 24V, J3 CAN_bus, J4 ENCODER, J5 ENCODER_POWER, J6 CONN_RS232, J7 M1 LIMIT UP DOWN, J8 Signal PWR, J9 MOTOR_OUT, Q1 2N3904, SW1 UP, SW2 DOWN, SW3 STOP, U1 MAX3232, U10 VNH5019A-E, U2 TSOP32S40F, U3 SN65HVD230, U4 ESP32-WROOM-32, U5 LM2596S-5, U6 AMS1117-3.3, U7 PC817, U8 PC817, U9 NCS1S1205SC

Commit message: fix schema ( fuse + annotation)
Parts:
- LED1: renamed from LED_GREEN_F3_POWER1; value LED -> LED_GREEN_F3
- LED2: renamed from LED_RED_F3_ERROR1; value LED_ERROR -> LED_RED_F3
- renumbered D3 to LED3
Changed lines of the file:
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@@
 	)
 	(junction
+		(at 137.16 187.96)
+		(diameter 0)
+		(color 0 0 0 0)
+	)
+	(junction
 		(at 166.37 154.94)
 		(diameter 0)
@@
 	(wire
 		(pts
-			(xy 137.16 187.96) (xy 147.32 187.96)
+			(xy 137.16 187.96) (xy 158.75 187.96)
 		)
 		(stroke
@@
 	(wire
 		(pts
-			(xy 158.75 187.96) (xy 158.75 191.77)
+			(xy 137.16 187.96) (xy 137.16 190.5)
 		)
 		(stroke
@@
 	(wire
 		(pts
-			(xy 152.4 187.96) (xy 147.32 187.96)
-		)
-		(stroke
-			(width 0)
-			(type default)
-		)
-	)
-	(wire
-		(pts
 			(xy 153.67 92.71) (xy 154.94 92.71)
 		)
@@
 	(wire
 		(pts
-			(xy 152.4 187.96) (xy 158.75 187.96)
-		)
-		(stroke
-			(width 0)
-			(type default)
-		)
-	)
-	(wire
-		(pts
 			(xy 171.45 176.53) (xy 171.45 180.34)
 		)
@@
 		(in_pos_files yes)
 		(dnp no)
-		(property "Reference" "LED_GREEN_F3_POWER1"
+		(property "Reference" "LED1"
 			(at 168.148 180.086 90)
 			(show_name no)
@@
 			)
 		)
-		(property "Value" "LED"
+		(property "Value" "LED_GREEN_F3"
 			(at 173.99 184.658 90)
 			(show_name no)
@@
 			)
 		)
-		(property "Description" ""
-			(at 171.45 184.15 0)
+		(property "Description" "LED_GREEN_F3_POWER"
+			(at 165.354 190.5 90)
 			(show_name no)
 			(do_not_autoplace no)
@@
 			(project "controller_Tv_Lift"
 				(path "/906b0219-e8e2-4a64-a5ea-d0350d472c53"
-					(reference "LED_GREEN_F3_POWER1")
+					(reference "LED1")
 					(unit 1)
 				)
@@
 		(lib_name "GND_15")
 		(lib_id "power:GND")
-		(at 158.75 191.77 0)
+		(at 137.16 190.5 0)
 		(unit 1)
 		(body_style 1)
@@
 		(dnp no)
 		(property "Reference" "#PWR028"
-			(at 158.75 198.12 0)
+			(at 137.16 196.85 0)
 			(hide yes)
 			(show_name no)
@@
 		)
 		(property "Value" "GND"
-			(at 155.702 191.77 0)
+			(at 134.112 190.5 0)
 			(show_name no)
 			(do_not_autoplace no)
@@
 		)
 		(property "Footprint" ""
-			(at 158.75 191.77 0)
+			(at 137.16 190.5 0)
 			(hide yes)
 			(show_name no)
@@
 		)
 		(property "Datasheet" ""
-			(at 158.75 191.77 0)
+			(at 137.16 190.5 0)
 			(hide yes)
 			(show_name no)
@@
 		)
 		(property "Description" ""
-			(at 158.75 191.77 0)
+			(at 137.16 190.5 0)
 			(show_name no)
 			(do_not_autoplace no)
@@
 		)
 		(property "Value" "150 uF 10V"
-			(at 159.004 189.484 0)
+			(at 159.004 178.562 0)
 			(show_name no)
 			(do_not_autoplace no)
@@
 		(in_pos_files yes)
 		(dnp no)
-		(property "Reference" "LED_RED_F3_ERROR1"
+		(property "Reference" "LED2"
 			(at 196.85 52.578 90)
 			(show_name no)
@@
 			)
 		)
-		(property "Value" "LED_ERROR"
+		(property "Value" "LED_RED_F3"
 			(at 205.74 43.688 90)
 			(show_name no)
@@
 			)
 		)
-		(property "Description" ""
+		(property "Description" "LED_RED_F3_ERROR1"
 			(at 203.2 43.18 0)
 			(show_name no)
@@
 			(project "controller_Tv_Lift"
 				(path "/906b0219-e8e2-4a64-a5ea-d0350d472c53"
-					(reference "LED_RED_F3_ERROR1")
+					(reference "LED2")
 					(unit 1)
 				)
@@
 		(in_pos_files yes)
 		(dnp no)
-		(property "Reference" "D3"
+		(property "Reference" "LED3"
 			(at 281.686 29.7052 90)
 			(show_name no)
@@
 			)
 		)
-		(property "Description" ""
+		(property "Description" "LED_Dual_Bidirectional_GREEN_BLUE"
 			(at 274.32 30.48 0)
 			(show_name no)
@@
 			(project "controller_Tv_Lift"
 				(path "/906b0219-e8e2-4a64-a5ea-d0350d472c53"
-					(reference "D3")
+					(reference "LED3")
 					(unit 1)
 				)
