File: hardware/TV_Lift_Kicad files/_autosave-controller_Tv_Lift.kicad_sch (KiCad schematic)
At the start: 102 parts, among them J1 socket LAN8720a, J10 1844210, J11 1844223, J12 C5360899, J2 1836189, J3 1844223, J4 1844210, J5 1844223, J6 1844223, J7 1844236, J8 C5360899, J9 1844210, Q2 MMBT3906, SW1 TS-1187A-BAB, SW2 TS-1187A-BAB, SW3 TS-1187A-BAB, SW4 TS-1187A-BAB, U1 MAX3232, U10 VNH5019A-E, U2 TSOP32S40F, U3 SN65HVD230, U4 ESP32-WROOM-32, U5 LM2596S-5, U6 AMS1117-3.3, U7 PC817, U8 PC817, U9 b0505s-1we

Commit message: change pins dry contavt and limit switch  and pwm
Connections:
- net DRY_CONTACT_DOWN: now also U4.6 (IO34); no longer U4.14 (IO12)
- net DRY_CONTACT_UP: now also U4.7 (IO35); no longer U4.16 (IO13)
- net M1_LIMIT_DOWN: now also U4.16 (IO13); no longer U4.7 (IO35)
- net M1_LIMIT_UP: now also U4.26 (IO4); no longer U4.6 (IO34)
- net M1_PWM: now also U4.14 (IO12); no longer U4.26 (IO4)
Changed lines of the file:
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@@
 	)
 	(label "M1_LIMIT_UP"
-		(at 115.57 87.63 0)
+		(at 115.57 41.91 0)
 		(effects
 			(font
@@
 	)
 	(label "M1_PWM"
-		(at 115.57 41.91 0)
+		(at 115.57 46.99 0)
 		(effects
 			(font
@@
 	)
 	(label "DRY_CONTACT_UP"
-		(at 115.57 49.53 0)
+		(at 115.57 90.17 0)
 		(effects
 			(font
@@
 	)
 	(label "DRY_CONTACT_DOWN"
-		(at 115.57 46.99 0)
+		(at 115.57 87.63 0)
 		(effects
 			(font
@@
 	)
 	(label "M1_LIMIT_DOWN"
-		(at 115.57 90.17 0)
+		(at 115.57 49.53 0)
 		(effects
 			(font
@@
 		(dnp no)
 		(property "Reference" "R26"
-			(at 130.556 85.09 90)
+			(at 130.302 80.264 90)
 			(show_name no)
 			(do_not_autoplace no)
@@
 		)
 		(property "Value" "470"
-			(at 130.302 80.01 90)
-			(show_name no)
-			(do_not_autoplace no)
+			(at 130.302 82.55 90)
+			(show_name no)
+			(do_not_autoplace no)
