File: hardware/TV_Lift_Kicad files/_autosave-controller_Tv_Lift.kicad_sch (KiCad schematic)
At the start: 103 parts, among them J1 socket LAN8720a, J10 1844210, J11 1844223, J12 C5360899, J2 1836189, J3 1844223, J4 1844210, J5 1844223, J6 1844223, J7 1844236, J8 C5360899, J9 1844210, Q2 C105432, SW1 TS-1187A-BAB, SW2 TS-1187A-BAB, SW3 TS-1187A-BAB, SW4 TS-1187A-BAB, U1 MAX3232, U10 VNH5019ATR-E, U2 C145345, U3 SN65HVD230, U4 ESP32-WROOM-32, U5 LM2596S-5, U6 AMS1117-3.3, U7 PC817, U8 PC817, U9 b0505s-1we

Commit message: fix BOM file and pcb
Parts:
- J1: value socket LAN8720a -> C54620381; footprint Connector_PinSocket_2.54mm:PinSocket_2x07_P2.54mm_Horizontal -> Connector_PinSocket_2.54mm:PinSocket_2x07_P2.54mm_Vertical
Changed lines of the file:
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@@
 			)
 		)
-		(property "Value" "socket LAN8720a"
+		(property "Value" "C54620381"
 			(at 41.91 153.416 0)
 			(show_name no)
@@
 			)
 		)
-		(property "Footprint" "Connector_PinSocket_2.54mm:PinSocket_2x07_P2.54mm_Horizontal"
+		(property "Footprint" "Connector_PinSocket_2.54mm:PinSocket_2x07_P2.54mm_Vertical"
 			(at 40.64 128.778 0)
 			(show_name no)
@@
 			)
 		)
-		(property "Description" ""
+		(property "Description" "socket LAN8720a"
 			(at 43.18 140.97 0)
 			(show_name no)
