File: hardware/TV_Lift_Kicad files/controller_Tv_Lift.kicad_sch (KiCad schematic)
At the start: 103 parts, among them J1 socket LAN8720a, J10 1844210, J11 1844223, J12 C5360899, J2 1836189, J3 1844223, J4 1844210, J5 1844223, J6 1844223, J7 1844236, J8 C5360899, J9 1844210, Q2 C105432, SW1 TS-1187A-BAB, SW2 TS-1187A-BAB, SW3 TS-1187A-BAB, SW4 TS-1187A-BAB, U1 MAX3232, U10 VNH5019ATR-E, U2 C145345, U3 SN65HVD230, U4 ESP32-WROOM-32, U5 LM2596S-5, U6 AMS1117-3.3, U7 PC817, U8 PC817, U9 b0505s-1we

Commit message: rewrite BOM
Parts:
- J1: value socket LAN8720a -> C54620381; footprint Connector_PinSocket_2.54mm:PinSocket_2x07_P2.54mm_Horizontal -> Connector_PinSocket_2.54mm:PinSocket_2x07_P2.54mm_Vertical
- LED2: value NCD0805R1 -> C84256
- U4: value ESP32-WROOM-32 -> ESP32-WROOM-32E-N16
Other:
- note added: "socket LAN8720a"
Changed lines of the file:
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@@
 	(generator_version "10.0")
 	(paper "A4")
+	(text "socket LAN8720a"
+		(exclude_from_sim no)
+		(at 43.18 156.718 0)
+		(effects
+			(font
+				(size 1.27 1.27)
+			)
+		)
+	)
 	(junction
 		(at 91.44 106.68)
@@
 			)
 		)
-		(property "Value" "ESP32-WROOM-32"
+		(property "Value" "ESP32-WROOM-32E-N16"
 			(at 104.648 97.536 0)
 			(show_name no)
@@
 			)
 		)
-		(property "Description" ""
+		(property "Description" "ESP32-WROOM-32E-N16"
 			(at 100.33 62.23 0)
 			(show_name no)
@@
 			)
 		)
-		(property "Value" "socket LAN8720a"
+		(property "Value" "C54620381"
 			(at 41.91 153.416 0)
 			(show_name no)
@@
 			)
 		)
-		(property "Footprint" "Connector_PinSocket_2.54mm:PinSocket_2x07_P2.54mm_Horizontal"
+		(property "Footprint" "Connector_PinSocket_2.54mm:PinSocket_2x07_P2.54mm_Vertical"
 			(at 40.64 128.778 0)
 			(show_name no)
@@
 			)
 		)
-		(property "Description" ""
+		(property "Description" "C54620381"
 			(at 43.18 140.97 0)
 			(show_name no)
@@
 			)
 		)
-		(property "Value" "NCD0805R1"
+		(property "Value" "C84256"
 			(at 198.12 35.814 0)
 			(show_name no)
@@
 			)
 		)
-		(property "Description" "Light emitting diode"
+		(property "Description" "Light emitting diode NCD0805R1"
 			(at 195.58 41.91 0)
 			(show_name no)
