File: hardware/TV_Lift_easy_Kicad files/Tv_Lift_easy.kicad_pcb (KiCad board)
At the start: 4 copper layers, 70 x 157.5 mm, 103 parts, among them J1 C54620381, J10 1844210, J11 1844223, J12 C5360899, J2 1836189, J3 1844223, J4 1844210, J5 1844223, J6 1844223, J7 1844236, J8 C5360899, J9 1844210, Q2 C105432, SW1 TS-1187A-BAB, SW2 TS-1187A-BAB, SW3 TS-1187A-BAB, SW4 TS-1187A-BAB, U1 MAX3232, U10 VNH5019ATR-E, U2 C145345, U3 SN65HVD230, U4 ESP32-WROOM-32, U5 LM2596S-5, U6 AMS1117-3.3, U7 PC817, U8 PC817, U9 b0505s-1we

Commit message: add  newe fuse easy board version
Parts:
- removed U7, U8: PC817, Package_DIP:DIP-4_W7.62mm
- removed U9: b0505s-1we, Converter_DCDC:Converter_DCDC_RECOM_R-78S-0.1_THT
- F1: value C5249699 -> C492610; footprint Fuse:Fuseholder_Blade_Mini_Keystone_3568 -> Fuse:Fuseholder_XF-506P_mini_blade_C492610
- LED2: value NCD0805R1 -> C84256
- U4: value ESP32-WROOM-32 -> ESP32-WROOM-32E-N16
- moved F1 4.74 mm to (68.5, 41.3)
- moved C20 1.55 mm to (95.0, 34.2)
- moved D1 1.52 mm to (88.6, 35.2)
- moved C21 1.50 mm to (102.5, 37.0)
Connections:
- J11 pad 2: /DRY_UP -> /DRY_CONTACT_UP
- J11 pad 3: /DRY_DOWN -> /DRY_CONTACT_DOWN
- J12 pad 1: /DRY_DOWN -> /DRY_CONTACT_DOWN
- J12 pad 2: /DRY_UP -> /DRY_CONTACT_UP
- R19 pad 1: Net-(U9-+VOUT) -> +5V
Routing:
- net Net-(U9--VOUT): track 23.2 -> 0.00 mm
- net /DRY_CONTACT_UP: track 86.2 -> 106.9 mm, vias 1 -> 2
- net /DRY_CONTACT_DOWN: track 94.3 -> 114.6 mm, vias 1 -> 2
- net /DRY_UP: track 13.1 -> 0.00 mm
- net /DRY_DOWN: track 12.7 -> 0.00 mm
- net +5V: track 204.5 -> 215.5 mm, vias 7 -> 8
- net Net-(U9-+VOUT): track 5.91 -> 0.00 mm
- net Net-(J9-M-): track 163.3 -> 166.7 mm
- net Net-(D1-A): track 30.3 -> 27.9 mm
- net +24V: track 77.3 -> 78.9 mm
- net Net-(J2-Pin_1): track 38.7 -> 38.0 mm
